File: ledBoard/LEDboard.sch (EAGLE design)
At the start: 107 parts

Commit message: added relay shield library and switching relay ino
Parts:
- added Q1: IRL7833, transistor-power:IRFZ48Z
- added U$1: PHOTON_SMD, Spark:PHOTON_SMD
Connections:
- net GND: now also U$1G$1.GND@2
- net VCC: now also U$1G$1.VIN
