File: relaySwitching/ledBoard/LEDboard.sch (EAGLE design)
At the start: 132 parts

Commit message: more schematics and code
Parts:
- removed R56: (no value), rcl:R-US_0204/2V
- added R61: 10K, resistor:R-US_0204/2V
- added R62, R63, R64, R65: 1K, rcl:R-US_0204/2V
- R57: value (none) -> 1K
- R58, R59, R60: value (none) -> 10K
Connections:
- new net N$262: R59.1, R62.1, T2.B
- new net N$263: R62.2, U$1G$1.D4
- new net N$264: R61.1, R64.1, T4.B
- new net N$265: R60.1, R63.1, T3.B
- net GND: now also R59.2, R60.2, R61.2; no longer T2.B, T3.B, T4.B
- net N$247: now also R63.2, U$1G$1.D5; no longer R59.1, R60.2
- net N$255: now also R64.2, U$1G$1.D6; no longer R60.1
- net N$258: now also U$1G$1.D3; no longer R59.2
- net N$261: now also R65.2; no longer R56.1
- net VCC: now also R65.1; no longer R56.2
Other:
- moved on the sheet: R59, R60

Commit message: more schematicz
Connections:
- new net NO: D1.A, D12.A, DZ1-1.A, DZ1-2.A, DZ11-4.A, DZ11-6.A, DZ12-2.A, DZ15-3.A, DZ15-5.A, DZ16-1.A, DZ16-2.A, DZ16-3.A, DZ16-4.A, DZ16-5.A, DZ26-1.A, DZ26-2.A
- net VCC: no longer D1.A, D12.A, DZ1-1.A, DZ1-2.A, DZ11-4.A, DZ11-6.A, DZ12-2.A, DZ15-3.A, DZ15-5.A, DZ16-1.A, DZ16-2.A, DZ16-3.A, DZ16-4.A, DZ16-5.A, DZ26-1.A, DZ26-2.A
Other:
- note added: "NO"
- note added: "VCC"
